File: pcb/RPiZero/pcb.kicad_sch (KiCad schematic)
At the start: 10 parts, among them M1 Vibration Motor, SW1 M2011S3AW03, U1 TP4056, U2 GENERIC_BUCK_CONV

Commit message: Add new folder for ESP32 PCB
Parts:
- removed M1: Vibration Motor, Connector_PinSocket_2.00mm:PinSocket_1x02_P2.00mm_Vertical, symbol Motor:Motor_DC
Changed lines of the file:
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@@
   (junction (at 157.48 102.87) (diameter 0) (color 0 0 0 0)
   )
-  (junction (at 144.78 58.42) (diameter 0) (color 0 0 0 0)
-  )
   (junction (at 154.94 97.79) (diameter 0) (color 0 0 0 0)
   )
   (junction (at 160.02 120.65) (diameter 0) (color 0 0 0 0)
   )
-  (junction (at 114.3 58.42) (diameter 0) (color 0 0 0 0)
-  )
   (junction (at 156.21 100.33) (diameter 0) (color 0 0 0 0)
   )
@@
     (stroke (width 0) (type default) (color 0 0 0 0))
   )
-  (wire (pts (xy 143.51 58.42) (xy 144.78 58.42))
-    (stroke (width 0) (type default) (color 0 0 0 0))
-  )
   (wire (pts (xy 153.67 69.85) (xy 99.06 69.85))
     (stroke (width 0) (type default) (color 0 0 0 0))
   )
-  (wire (pts (xy 144.78 46.99) (xy 144.78 58.42))
-    (stroke (width 0) (type default) (color 0 0 0 0))
-  )
   (wire (pts (xy 130.81 142.24) (xy 130.81 146.05))
     (stroke (width 0) (type default) (color 0 0 0 0))
@@
     (stroke (width 0) (type default) (color 0 0 0 0))
   )
-  (wire (pts (xy 135.89 46.99) (xy 144.78 46.99))
-    (stroke (width 0) (type default) (color 0 0 0 0))
-  )
   (wire (pts (xy 63.5 91.44) (xy 25.4 91.44))
     (stroke (width 0) (type default) (color 0 0 0 0))
@@
     (stroke (width 0) (type default) (color 0 0 0 0))
   )
-  (wire (pts (xy 114.3 46.99) (xy 114.3 58.42))
-    (stroke (width 0) (type default) (color 0 0 0 0))
-  )
   (wire (pts (xy 91.44 100.33) (xy 91.44 157.48))
     (stroke (width 0) (type default) (color 0 0 0 0))
@@
     (stroke (width 0) (type default) (color 0 0 0 0))
   )
-  (wire (pts (xy 123.19 46.99) (xy 114.3 46.99))
-    (stroke (width 0) (type default) (color 0 0 0 0))
-  )
   (wire (pts (xy 149.86 74.93) (xy 149.86 80.01))
     (stroke (width 0) (type default) (color 0 0 0 0))
@@
     (stroke (width 0) (type default) (color 0 0 0 0))
   )
-  (wire (pts (xy 96.52 58.42) (xy 114.3 58.42))
+  (wire (pts (xy 96.52 58.42) (xy 119.38 58.42))
     (stroke (width 0) (type default) (color 0 0 0 0))
   )
@@
     (stroke (width 0) (type default) (color 0 0 0 0))
   )
-  (wire (pts (xy 114.3 58.42) (xy 119.38 58.42))
-    (stroke (width 0) (type default) (color 0 0 0 0))
-  )
   (wire (pts (xy 135.89 139.7) (xy 156.21 139.7))
     (stroke (width 0) (type default) (color 0 0 0 0))
   )
-  (wire (pts (xy 144.78 58.42) (xy 152.4 58.42))
+  (wire (pts (xy 143.51 58.42) (xy 152.4 58.42))
     (stroke (width 0) (type default) (color 0 0 0 0))
   )
@@
     )
     (pin "1")
+    (pin "2")
     (pin "3")
     (pin "4")
     (pin "5")
     (pin "6")
-    (pin "2")
   )
   (symbol (lib_id "Connector:Conn_01x05_Female") (at 177.8 100.33 0) (mirror x) (unit 1)
@@
     (pin "2")
   )
-  (symbol (lib_id "Motor:Motor_DC") (at 128.27 46.99 90) (unit 1)
-    (in_bom yes) (on_board yes) (fields_autoplaced)
-    (property "Reference" "M1" (id 0) (at 130.81 38.1 90))
-    (property "Value" "Vibration Motor" (id 1) (at 130.81 40.64 90))
-    (property "Footprint" "Connector_PinSocket_2.00mm:PinSocket_1x02_P2.00mm_Vertical" (id 2) (at 130.556 46.99 0)
-      (effects (font (size 1.27 1.27)) hide)
-    )
-    (property "Datasheet" "~" (id 3) (at 130.556 46.99 0)
-      (effects (font (size 1.27 1.27)) hide)
-    )
-    (pin "1")
-    (pin "2")
-  )
   (symbol (lib_id "getting_started:M2011S3AW03") (at 53.34 81.28 0) (unit 1)
     (in_bom yes) (on_board yes) (fields_autoplaced)
@@
       (reference "D1") (unit 1) (value "LED") (footprint "LED_THT:LED_D3.0mm")
     )
-    (path "/60b6144a-b98b-4982-931d-771d6c77092f"
-      (reference "M1") (unit 1) (value "Vibration Motor") (footprint "Connector_PinSocket_2.00mm:PinSocket_1x02_P2.00mm_Vertical")
-    )
     (path "/c93902f3-b47f-45aa-b82f-90ec417421e6"
